File: photos/co2 timer v2.kicad_sch (KiCad schematic)
At the start: 23 parts, among them J1 9V_BATT_IN, J2 SOLENOID_OUT, J3 ICSP, J4 TM1637_DISPLAY, Q1 IRL540NPBF, SW1 UP, SW2 SET, U1 ATtiny85-20PU, U2 DS3231SN, U3 AMS1117-3.3

Commit message: Sync deployed GreenGuard web app state to git
Snapshot of deployed-but-uncommitted work that had accumulated in the
working tree (the reason fixes kept appearing 'lost' each session):
- 92 modified files (app/pages, app/lib, app/components, astro/src, etc.)
- 28 new deployed API endpoints (admin data routes, book/slots,
  cron/ads-tracking-health, gbp-post/reply, etc.) + design-sync styles
- remove dead app/lib/gnl.js

Excludes: build artifacts (app/dist, ds-bundle, design-sync), the
unrelated Cooling_Tower Ignition project files, and the other session's
astro/public prototype binaries.
Parts:
- added R7: 4K7, Resistor_SMD:R_0805_2012Metric, symbol Device:R
Changed lines of the file:
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@@
     (property "Footprint" "Resistor_SMD:R_0805_2012Metric" (at 150 62 0))
+  )
+  (symbol (lib_id "Device:R") (at 162 55 0) (unit 1)
+    (property "Reference" "R7" (at 162 50 0))
+    (property "Value" "4K7" (at 162 60 0))
+    (property "Footprint" "Resistor_SMD:R_0805_2012Metric" (at 162 62 0))
+    (property "Description" "I2C SCL pullup — PB1/SCL to VCC" (at 162 64 0))
   )
   (symbol (lib_id "Device:R") (at 150 70 0) (unit 1)
@@
     (property "Footprint" "Connector_PinHeader_2.54mm:PinHeader_2x03_P2.54mm_Vertical" (at 55 110 0))
   )
+  ;; ── R7 VCC power symbol (top of SCL pullup) ─────────────
+  (symbol (lib_id "power:VCC") (at 162 47 0) (unit 1)
+    (property "Reference" "#PWR04" (at 162 51 0))
+    (property "Value" "+3V3" (at 162 44 0))
+  )
   ;; ── Net Labels ───────────────────────────────────────────
   (label "TM1637_CLK" (at 92 62 0))
@@
   (label "SDA" (at 153 62 0))
   (label "SCL" (at 153 65 0))
+  (label "SCL" (at 165 62 0))
   (label "RTC_INT" (at 153 68 0))
   (label "VBAT_3V3" (at 153 71 0))
